Commit message: Added Dock
 Dock and Astrobee positions are not accurate

File: Assets/Urdf/astrobee_dock/model.urdf (robot description, URDF)
Before this commit: robot handrail, 1 links, 0 joints
Links:
- link body: geometry collision mesh filename=package://astrobee_dock/meshes/dock_base.dae; visual mesh filename=package://astrobee_dock/meshes/dock_base.dae
